Commit message: URDF visualization working with joint state publisher

File: urdf/kortex-gen3-lite.urdf (robot description, URDF)
Before this commit: robot kortex-arm, 4 links, 3 joints
Links:
- added link forearm_link; visual mesh filename=package://kortex-gen3-lite_description/meshes/forearm_link.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 scale=1.0 1.0 1.0
- added link lower_wrist_link; visual mesh filename=package://kortex-gen3-lite_description/meshes/lower_wrist_l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 scale=1.0 1.0 1.0
- added link upper_wrist_link; visual mesh filename=package://kortex-gen3-lite_description/meshes/upper_wrist_l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 scale=1.0 1.0 1.0
Joints:
- added joint arm_to_forearm_joint: type revolute, parent arm_link, child forearm_link, origin xyz=0 0.28 0.01 rpy=0 3.140 3.140, axis 0.0 0.0 1.0, limit lower=-3.14 upper=3.14 effort=0.0 velocity=0.0
- added joint forearm_to_lower_wrist_joint: type revolute, parent forearm_link, child lower_wrist_link, origin xyz=0 -0.139 0.02 rpy=1.571 -1.571 0, axis 0.0 0.0 1.0, limit lower=-3.14 upper=3.14 effort=0.0 velocity=0.0
- added joint lower_wrist_to_upper_wrist_joint: type revolute, parent lower_wrist_link, child upper_wrist_link, origin xyz=0.028 0.0 0.105 rpy=0 1.571 0, axis 0.0 0.0 1.0, limit lower=-3.14 upper=3.14 effort=0.0 velocity=0.0
- joint shoulder_to_arm_joint: axis (none) -> 0.0 0.0 1.0; limit (none) -> lower=-3.14 upper=3.14 effort=0.0 velocity=0.0; type fixed -> revolute
